File: sepiapcb/sepiapcb2/sepiapcb2.sch (KiCad schematic (older format))
At the start: 5 parts, among them SW1 SW_DPDT_x2

Commit message: Enlarged sepia almost done
Parts:
- D3, D4: footprint LED_SMD:LED_1206_3216Metric_Pad1.42x1.75mm_HandSolder -> sepiapcb:LED_1206_3216Metric_ReverseMount_NoHole1.8x2.4mm
Changed lines of the file:
@@
 F 0 "D4" H 5343 2716 50  0000 C CNN
 F 1 "LED" H 5343 2625 50  0000 C CNN
-F 2 "LED_SMD:LED_1206_3216Metric_Pad1.42x1.75mm_HandSolder" H 5350 2500 50  0001 C CNN
+F 2 "sepiapcb:LED_1206_3216Metric_ReverseMount_NoHole1.8x2.4mm" H 5350 2500 50  0001 C CNN
 F 3 "~" H 5350 2500 50  0001 C CNN
 	1    5350 2500
@@
 F 0 "D3" H 4993 2716 50  0000 C CNN
 F 1 "LED" H 4993 2625 50  0000 C CNN
-F 2 "LED_SMD:LED_1206_3216Metric_Pad1.42x1.75mm_HandSolder" H 5000 2500 50  0001 C CNN
+F 2 "sepiapcb:LED_1206_3216Metric_ReverseMount_NoHole1.8x2.4mm" H 5000 2500 50  0001 C CNN
 F 3 "~" H 5000 2500 50  0001 C CNN
 	1    5000 2500
