File: sepiapcb/sepiapcb2/sepiapcb2.kicad_pcb (KiCad board)
At the start: 2 copper layers, 98.1 x 75.2 mm, 5 parts, among them SW1 SW_DPDT_x2

Commit message: Fixe signature -> a curved one didn't work
Other:
- board text added: "https://josefadamcik.cz"

Commit message: Adde pads for pins, gerebre files
Parts:
- added REF**: brooch_pin_pad, sepiapcb:brooch_pin_pad, B.Cu at (62.9, 54.4)
- added REF**: brooch_pin_pad, sepiapcb:brooch_pin_pad, B.Cu at (81.1, 77.4)
- added REF**: brooch_pin_pad, sepiapcb:brooch_pin_pad, B.Cu at (89.6, 56.0)
Other:
- board text added: "+"
- board text added: "@josefadamcik"
- board text added: "D1"
- board text added: "D2"
Changed lines of the file:
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@@
   (general
     (thickness 1.6)
-    (drawings 184)
+    (drawings 189)
     (tracks 34)
     (zones 0)
-    (modules 5)
+    (modules 8)
     (nets 4)
   )
@@
   (layers
     (0 F.Cu signal hide)
-    (31 B.Cu signal hide)
+    (31 B.Cu signal)
     (32 B.Adhes user hide)
     (33 F.Adhes user hide)
-    (34 B.Paste user hide)
+    (34 B.Paste user)
     (35 F.Paste user hide)
     (36 B.SilkS user)
     (37 F.SilkS user hide)
-    (38 B.Mask user hide)
+    (38 B.Mask user)
     (39 F.Mask user hide)
     (40 Dwgs.User user hide)
@@
     (44 Edge.Cuts user)
     (45 Margin user hide)
-    (46 B.CrtYd user hide)
+    (46 B.CrtYd user)
     (47 F.CrtYd user hide)
-    (48 B.Fab user hide)
+    (48 B.Fab user)
     (49 F.Fab user hide)
   )
@@
     (add_net "Net-(D1-Pad1)")
   )
+  (module sepiapcb:brooch_pin_pad (layer B.Cu)
+    (at 62.9031 54.356)
+    (fp_text reference REF** (at 0.508 4.826) (layer B.SilkS) hide
+      (effects (font (size 1 1) (thickness 0.15)) (justify mirror))
+    )
+    (fp_text value brooch_pin_pad (at 0.254 -4.826) (layer B.Fab)
+      (effects (font (size 1 1) (thickness 0.15)) (justify mirror))
+    )
+    (fp_circle (center 0 0) (end 5.75 0) (layer Dwgs.User) (width 0.12))
+    (pad 1 smd circle (at 0 0) (size 8 8) (layers B.Cu B.Paste B.Mask))
+  )
+  (module sepiapcb:brooch_pin_pad (layer B.Cu)
+    (at 81.0768 77.3938)
+    (fp_text reference REF** (at 0.508 4.826) (layer B.SilkS) hide
+      (effects (font (size 1 1) (thickness 0.15)) (justify mirror))
+    )
+    (fp_text value brooch_pin_pad (at 0.254 -4.826) (layer B.Fab)
+      (effects (font (size 1 1) (thickness 0.15)) (justify mirror))
+    )
+    (fp_circle (center 0 0) (end 5.75 0) (layer Dwgs.User) (width 0.12))
+    (pad 1 smd circle (at 0 0) (size 8 8) (layers B.Cu B.Paste B.Mask))
+  )
+  (module sepiapcb:brooch_pin_pad (layer B.Cu)
+    (at 89.5858 56.007)
+    (fp_text reference REF** (at 0.508 4.826) (layer B.SilkS) hide
+      (effects (font (size 1 1) (thickness 0.15)) (justify mirror))
+    )
+    (fp_text value brooch_pin_pad (at 0.254 -4.826) (layer B.Fab) hide
+      (effects (font (size 1 1) (thickness 0.15)) (justify mirror))
+    )
+    (fp_circle (center 0 0) (end 5.75 0) (layer Dwgs.User) (width 0.12))
+    (pad 1 smd circle (at 0 0) (size 8 8) (layers B.Cu B.Paste B.Mask))
+  )
   (module sepiapcb:LED_1206_3216Metric_ReverseMount_NoHole1.8x2.4mm (layer B.Cu)
     (at 75.184 55.2196)
@@
     (tags "diode reverse")
     (attr smd)
-    (fp_text reference D4 (at 0 2.145) (layer B.SilkS)
+    (fp_text reference D4 (at -0.1143 -2.7051) (layer B.SilkS)
       (effects (font (size 1 1) (thickness 0.15)) (justify mirror))
     )
-    (fp_text value LED (at 0 -2.145) (layer B.Fab)
+    (fp_text value LED (at 0.127 -2.5908) (layer B.Fab) hide
       (effects (font (size 1 1) (thickness 0.15)) (justify mirror))
     )
     (fp_circle (center 0 0) (end 0.4 0) (layer B.Mask) (width 0.9))
-    (fp_text user %R (at 0 0) (layer B.Fab)
+    (fp_text user %R (at 0.0254 -2.5908) (layer B.Fab)
       (effects (font (size 0.8 0.8) (thickness 0.12)) (justify mirror))
     )
@@
     (tags "diode reverse")
     (attr smd)
-    (fp_text reference D3 (at 0 2.145) (layer B.SilkS)
+    (fp_text reference D3 (at 0.0762 2.9972) (layer B.SilkS)
       (effects (font (size 1 1) (thickness 0.15)) (justify mirror))
     )
-    (fp_text value LED (at 0 -2.145) (layer B.Fab)
+    (fp_text value LED (at 0 -2.145) (layer B.Fab) hide
       (effects (font (size 1 1) (thickness 0.15)) (justify mirror))
     )
     (fp_circle (center 0 0) (end 0.4 0) (layer B.Mask) (width 0.9))
-    (fp_text user %R (at 0 0) (layer B.Fab)
+    (fp_text user %R (at -0.0889 -2.5781) (layer B.Fab)
       (effects (font (size 0.8 0.8) (thickness 0.12)) (justify mirror))
     )
@@
     (descr "Ultraminiature Surface Mount Slide Switch")
     (attr smd)
-    (fp_text reference SW1 (at 0 3.2 35) (layer B.SilkS)
+    (fp_text reference SW1 (at 6.06571 -0.248857 125) (layer B.SilkS)
       (effects (font (size 1 1) (thickness 0.15)) (justify mirror))
     )
-    (fp_text value SW_DPDT_x2 (at 0 -4.25 35) (layer B.Fab)
+    (fp_text value SW_DPDT_x2 (at 0 -4.25 35) (layer B.Fab) hide
       (effects (font (size 1 1) (thickness 0.15)) (justify mirror))
     )
@@
     (fp_line (start -1.4 -2.95) (end -1.2 -3.15) (layer B.Fab) (width 0.1))
     (fp_line (start -1.4 -1.65) (end -1.4 -2.95) (layer B.Fab) (width 0.1))
-    (fp_text user %R (at 0 3.2 35) (layer B.Fab)
+    (fp_text user %R (at 5.992866 -0.144825 125) (layer B.Fab)
       (effects (font (size 1 1) (thickness 0.15)) (justify mirror))
     )
@@
       (effects (font (size 1 1) (thickness 0.15)) (justify mirror))
     )
-    (fp_text value Battery_Cell (at 10.499999 11.6 310) (layer B.Fab)
+    (fp_text value Battery_Cell (at 9.93497 8.253537 310) (layer B.Fab)
       (effects (font (size 1 1) (thickness 0.15)) (justify mirror))
     )
@@
       (net 2 +3V0))
   )
-  (gr_text https://josefadamcik.cz (at 88.0364 75.8698) (layer B.SilkS)
+  (gr_text @josefadamcik (at 43.5864 74.3204 40) (layer B.SilkS)
+    (effects (font (size 1 1) (thickness 0.15)) (justify mirror))
+  )
+  (gr_text D2 (at 73.406 69.9643) (layer B.SilkS)
+    (effects (font (size 1 1) (thickness 0.15)) (justify mirror))
+  )
+  (gr_text D1 (at 65.5828 61.9379) (layer B.SilkS)
+    (effects (font (size 1 1) (thickness 0.15)) (justify mirror))
+  )
+  (gr_text + (at 75.2983 65.6717) (layer B.SilkS)
+    (effects (font (size 1 1) (thickness 0.15)) (justify mirror))
+  )
+  (gr_text + (at 69.8119 60.2996) (layer B.SilkS)
+    (effects (font (size 1 1) (thickness 0.15)) (justify mirror))
+  )
+  (gr_text https://josefadamcik.cz (at 60.7187 81.8388 40) (layer B.SilkS)
     (effects (font (size 1.5 1.5) (thickness 0.3)) (justify mirror))
   )
@@
     (polygon
       (pts
-        (xy 83.312 61.6966) (xy 83.312 65.4558) (xy 77.9018 65.3034) (xy 78.0034 61.6204)
+        (xy 83.312 61.6966) (xy 83.4009 64.9351) (xy 77.9272 65.0875) (xy 77.9907 61.7855)
       )
     )
