File: sepiapcb/sepiapcb2.sch (KiCad schematic (older format))
At the start: 5 parts, among them SW1 SW_DPDT_x2

Commit message: PCB with THT tentacles
Parts:
- D1: footprint sepiapcb:sepia_footprint_enlarged_pcb -> sepiapcb:sepia_footprint_enlarged_thttent_pcb
Changed lines of the file:
@@
 F 0 "D1" V 4500 2050 50  0000 L CNN
 F 1 "LED_Dual_AACC" V 4600 1700 50  0000 L CNN
-F 2 "sepiapcb:sepia_footprint_enlarged_pcb" H 4330 2400 50  0001 C CNN
+F 2 "sepiapcb:sepia_footprint_enlarged_thttent_pcb" H 4330 2400 50  0001 C CNN
 F 3 "~" H 4330 2400 50  0001 C CNN
 	1    4300 2400
