File: sepiapcb/sepiapcb2.kicad_pcb (KiCad board)
At the start: 2 copper layers, 98.1 x 75.2 mm, 8 parts, among them SW1 SW_DPDT_x2

Commit message: PCB with THT tentacles
Parts:
- D1: footprint sepiapcb:sepia_footprint_enlarged_pcb -> sepiapcb:sepia_footprint_enlarged_thttent_pcb
Connections:
- SW1 pad 3: (no net) -> Net-(SW1-Pad3)
Routing:
- net Net-(D1-Pad1): track 36.0 -> 54.1 mm
- net GND: track 28.1 -> 18.0 mm

Commit message: Gerber fiele
Parts:
- renumbered REF** to PIN
Changed lines of the file:
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@@
   (page A4)
   (layers
-    (0 F.Cu signal hide)
+    (0 F.Cu signal)
     (31 B.Cu signal)
-    (32 B.Adhes user hide)
-    (33 F.Adhes user hide)
+    (32 B.Adhes user)
+    (33 F.Adhes user)
     (34 B.Paste user)
-    (35 F.Paste user hide)
+    (35 F.Paste user)
     (36 B.SilkS user)
-    (37 F.SilkS user hide)
+    (37 F.SilkS user)
     (38 B.Mask user)
-    (39 F.Mask user hide)
-    (40 Dwgs.User user hide)
-    (41 Cmts.User user hide)
-    (42 Eco1.User user hide)
-    (43 Eco2.User user hide)
+    (39 F.Mask user)
+    (40 Dwgs.User user)
+    (41 Cmts.User user)
+    (42 Eco1.User user)
+    (43 Eco2.User user)
     (44 Edge.Cuts user)
-    (45 Margin user hide)
+    (45 Margin user)
     (46 B.CrtYd user)
-    (47 F.CrtYd user hide)
+    (47 F.CrtYd user)
     (48 B.Fab user)
-    (49 F.Fab user hide)
+    (49 F.Fab user)
   )
   (setup
@@
   (module sepiapcb:brooch_pin_pad (layer B.Cu)
     (at 64 53.5)
-    (fp_text reference REF** (at 0.508 4.826) (layer B.SilkS)
+    (fp_text reference PIN (at 5.34 2.09) (layer B.SilkS)
       (effects (font (size 1 1) (thickness 0.15)) (justify mirror))
     )
@@
   (module sepiapcb:brooch_pin_pad (layer B.Cu)
     (at 89.5 55.5)
-    (fp_text reference REF** (at 0.508 4.826) (layer B.SilkS)
+    (fp_text reference PIN (at 5.79 0.72) (layer B.SilkS)
       (effects (font (size 1 1) (thickness 0.15)) (justify mirror))
     )
